Commit message: init

File: autorally_description/urdf/autoRallyPlatform.urdf.xacro (robot description, xacro)
@@ -347,4 +347,5 @@
     <child link="chassis"/>
   </joint>
+<!--
   <link name="imu_link">
     <collision>
@@ -371,6 +372,7 @@
     <child link="camera_link"/>
   </joint>
+-->
   <!-- Camera -->
-  <link name="camera_link">
+<!--  <link name="camera_link">
     <collision>
       <origin xyz="0 0 0" rpy="0 0 0"/>
@@ -378,5 +380,5 @@
     <box size="0.02 0.02 0.02"/>
       </geometry>
-    </collision>
+    </collision>-->
 <!--
     <visual>
@@ -388,5 +390,5 @@
     </visual>
 -->
-    <inertial>
+ <!--   <inertial>
       <mass value="1e-5" />
       <origin xyz="0 0 0" rpy="0 0 0"/>
@@ -400,6 +402,7 @@
     <child link="side_camera_link"/>
   </joint>
+-->
   <!-- Camera -->
-  <link name="side_camera_link">
+ <!-- <link name="side_camera_link">-->
     <!-- <collision>
       <origin xyz="0 0 0" rpy="0 0 0"/>
@@ -416,12 +419,55 @@
     </visual>
     -->
-    <inertial>
+<!--    <inertial>
       <mass value="1e-5" />
       <origin xyz="0 0 0" rpy="0 0 0"/>
       <inertia ixx="1e-6" ixy="0" ixz="0" iyy="1e-6" iyz="0" izz="1e-6" />
     </inertial>
-  </link>
+  </link>-->
+<link name = "laser_link">
+  <inertial>
+    <mass value = "1e-5"/>
+    <inertia ixx="1e-6" ixy="0" ixz="0" iyy="1e-6" iyz="0" izz="1e-6" />
+  </inertial>
+</link>
+ <joint name = "laser_joint" type = "fixed">
+    <axis xyz="0 0 0" />
+    <origin xyz="0 0 0.25" rpy="0 0 0"/>
+    <parent link="base_link"/>
+    <child link="laser_link"/>
+  </joint>
+<gazebo reference = "laser_link">
+  <sensor name = "laser_sensor" type = 'ray'>
+    <ray>
+      <scan>
+        <horizontal>
+          <samples>360</samples>
+          <resolution>1</resolution>
+          <min_angle>-3.14</min_angle>
+          <max_angle>3.14</max_angle>
+        </horizontal>
+        <vertical>
+          <samples>1</samples>
+          <min_angle>-0.1</min_angle>
+          <max_angle>-0.35</max_angle>
+        </vertical>
+      </scan>
+      <range>
+        <min>0.3</min>
+        <max>25</max>
+        <resolution>0.01</resolution>
+      </range>
+    </ray>
+    <plugin name = 'laser' filename = 'libgazebo_ros_laser.so'>
+      <topicName>/ytscan</topicName>
+      <frameName>laser_link</frameName>
+    </plugin>
+    <always_on>1</always_on>
+    <update_rate>30</update_rate>
+    <visualize>1</visualize>
+  </sensor>
+</gazebo>
   <!-- camera -->
-  <gazebo reference="camera_link">
+ <!-- <gazebo reference="camera_link">
     <sensor type="multicamera" name="stereo_camera">
       <update_rate>30.0</update_rate>
@@ -468,7 +514,7 @@
         <imageTopicName>image_raw</imageTopicName>
         <cameraInfoTopicName>camera_info</cameraInfoTopicName>
-        <frameName>left_camera_optical_frame</frameName>
+        <frameName>left_camera_optical_frame</frameName>-->
         <!--<rightFrameName>right_camera_optical_frame</rightFrameName>-->
-        <hackBaseline>0.14</hackBaseline>
+        <!--<hackBaseline>0.14</hackBaseline>-->
         <!-- <distortionK1>-0.212652</distortionK1>
         <distortionK2>0.085434</distortionK2>
@@ -476,9 +522,9 @@
         <distortionT1>-0.000336</distortionT1>
         <distortionT2>0.0</distortionT2> -->
-      </plugin>
+<!--      </plugin>
     </sensor>
-  </gazebo>
+  </gazebo>-->
    <!-- camera -->
-  <gazebo reference="side_camera_link">
+<!--  <gazebo reference="side_camera_link">
     <sensor type="camera" name="camera_side">
       <update_rate>30.0</update_rate>
@@ -495,9 +541,9 @@
         </clip>
         <noise>
-          <type>gaussian</type>
+          <type>gaussian</type>-->
           <!-- Noise is sampled independently per pixel on each frame.
                That pixel's noise value is added to each of its color
                channels, which at that point lie in the range [0,1]. -->
-          <mean>0.0</mean>
+  <!--        <mean>0.0</mean>
           <stddev>0.007</stddev>
         </noise>
@@ -510,5 +556,5 @@
         <cameraInfoTopicName>camera_info</cameraInfoTopicName>
         <frameName>side_camera_link</frameName>
-        <hackBaseline>0.07</hackBaseline>
+        <hackBaseline>0.07</hackBaseline>-->
         <!-- <distortionK1>0.0</distortionK1>
         <distortionK2>0.0</distortionK2>
@@ -516,7 +562,8 @@
         <distortionT1>0.0</distortionT1>
         <distortionT2>0.0</distortionT2> -->
-      </plugin>
+<!--      </plugin>
     </sensor>
   </gazebo>
+-->
   <!-- Wheels -->
   <xacro:front_wheel lr_prefix="left" fr_prefix="front"
@@ -545,5 +592,5 @@
       <robotSimType>gazebo_ros_control/DefaultRobotHWSim</robotSimType>
     </plugin>
-    <plugin name="imu" filename="libhector_gazebo_ros_imu.so">
+ <!--   <plugin name="imu" filename="libhector_gazebo_ros_imu.so">
       <robotNamespace>/autorally_platform</robotNamespace>
       <serviceName>/imu/calibrate</serviceName>
@@ -578,5 +625,5 @@
       <velocityDrift>0 0 0</velocityDrift>
       <velocityGaussianNoise>0.005 0.005 0.05</velocityGaussianNoise>
-    </plugin>
+    </plugin>-->
     <!-- <plugin name="tire_friction" filename="libTireFrictionPlugin.so">
       <link_name>left_rear_wheel</link_name>
